Commit message: Cleaned the code, added parameters

File: models/double_rock_pbr/pbr_mesh.urdf (robot description, URDF)
Before this commit: robot pbr_mesh, 1 links, 0 joints
Links:
- link base_link: mass 1437.596 -> 0.105; geometry collision mesh filename=file:///home/akshay/mesh_files/sacled_2.obj scale=1.0 1.0 1.0; visual mesh filename=file:///home/akshay/mesh_files/sacled_2.obj scale=1.0 1.0 1.0
