Commit message: Made chnages in the launch file according to the sim

File: models/SP2_PBRmodel/sp2.urdf (robot description, URDF)
Before this commit: robot sp2_robot, 1 links, 0 joints
Links:
- link base_link: geometry collision mesh filename=file:///home/akshay/ros2_ws/src/virtual_shake_robot_pybulle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 scale=1.0 1.0 1.0; visual mesh filename=file:///home/akshay/ros2_ws/src/virtual_shake_robot_pybulle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 scale=1.0 1.0 1.0
