Commit message: suggested chnages the path and inertia confirmed

File: models/SP1_PBRmodel/sp1.urdf (robot description, URDF)
Before this commit: robot sp1_robot, 1 links, 0 joints
Links:
- link base_link: geometry collision mesh filename=package://virtual_shake_robot_pybullet/models/SP1_PBRmodel/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 scale=1.0 1.0 1.0; visual mesh filename=package://virtual_shake_robot_pybullet/models/SP1_PBRmodel/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 scale=1.0 1.0 1.0

File: models/double_rock_pbr/pbr_mesh.urdf (robot description, URDF)
Before this commit: robot pbr_mesh, 1 links, 0 joints
Links:
- link base_link: mass 0.105 -> 1437.596; geometry collision mesh filename=package://virtual_shake_robot_pybullet/models/double_rock_p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 scale=1.0 1.0 1.0; visual mesh filename=package://virtual_shake_robot_pybullet/models/double_rock_p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 scale=1.0 1.0 1.0

Commit message: Addressed the chnages

File: models/SP1_PBRmodel/sp1.urdf (robot description, URDF)
Before this commit: robot sp1_robot, 1 links, 0 joints
Links:
- link base_link: geometry collision mesh filename=package://src/virtual_shake_robot_pybullet/models/SP1_PBRmo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 scale=1.0 1.0 1.0; visual mesh filename=package://src/virtual_shake_robot_pybullet/models/SP1_PBRmo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 scale=1.0 1.0 1.0

Commit message: removed rolling friction and other chnages

File: models/SP1_PBRmodel/sp1.urdf (robot description, URDF)
Before this commit: robot sp1_robot, 1 links, 0 joints
Links:
- link base_link: geometry collision mesh filename=package://virtual_shake_robot_pybullet/models/SP1_PBRmodel/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 scale=1.0 1.0 1.0; visual mesh filename=package://virtual_shake_robot_pybullet/models/SP1_PBRmodel/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 scale=1.0 1.0 1.0

Commit message: range singe_recording
Chnages in control_node.py

Chnages the random seed generation

Implemented the earthquake_batch

earthquake_parser.py

 Final_structure for earthquake-batch

Changes in the callback function

Chnages

Changes in the single_recording_range

Chnages in the callback

Chnages in the functionlity

all the chnages

File: models/SP1_PBRmodel/sp1.urdf (robot description, URDF)
Before this commit: robot sp1_robot, 1 links, 0 joints
Links:
- link base_link: geometry collision mesh filename=package://virtual_shake_robot_pybullet/models/SP1_PBRmodel/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 scale=1 1 1; visual mesh filename=package://virtual_shake_robot_pybullet/models/SP1_PBRmodel/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 scale=1 1 1
